File: IOB-Adapter-Generic_array.brd (EAGLE design)
At the start: 106.7 x 104.1 mm, 53 parts

Commit message: added values for connectors
Parts:
- CARRIER: value (none) -> 10x10
- FID-LR, FID-UL: value (none) -> FIDUCIAL
Changed lines of the file:
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@@
 <grid distance="50" unitdist="mil" unit="mil" style="dots" multiple="2" display="yes" altdistance="25" altunitdist="mil" altunit="mil"/>
 <layers>
-<layer number="1" name="Top" color="4" fill="1" visible="no" active="yes"/>
+<layer number="1" name="Top" color="4" fill="1" visible="yes" active="yes"/>
 <layer number="2" name="Route2" color="1" fill="3" visible="no" active="no"/>
 <layer number="3" name="Route3" color="4" fill="3" visible="no" active="no"/>
@@
 <layer number="19" name="Unrouted" color="6" fill="1" visible="yes" active="yes"/>
 <layer number="20" name="Dimension" color="15" fill="1" visible="yes" active="yes"/>
-<layer number="21" name="tPlace" color="7" fill="1" visible="no" active="yes"/>
-<layer number="22" name="bPlace" color="7" fill="1" visible="yes" active="yes"/>
-<layer number="23" name="tOrigins" color="15" fill="1" visible="no" active="yes"/>
-<layer number="24" name="bOrigins" color="15" fill="1" visible="yes" active="yes"/>
-<layer number="25" name="tNames" color="7" fill="1" visible="no" active="yes"/>
-<layer number="26" name="bNames" color="7" fill="1" visible="yes" active="yes"/>
-<layer number="27" name="tValues" color="7" fill="1" visible="no" active="yes"/>
-<layer number="28" name="bValues" color="7" fill="1" visible="yes" active="yes"/>
+<layer number="21" name="tPlace" color="7" fill="1" visible="yes" active="yes"/>
+<layer number="22" name="bPlace" color="7" fill="1" visible="no" active="yes"/>
+<layer number="23" name="tOrigins" color="15" fill="1" visible="yes" active="yes"/>
+<layer number="24" name="bOrigins" color="15" fill="1" visible="no" active="yes"/>
+<layer number="25" name="tNames" color="7" fill="1" visible="yes" active="yes"/>
+<layer number="26" name="bNames" color="7" fill="1" visible="no" active="yes"/>
+<layer number="27" name="tValues" color="7" fill="1" visible="yes" active="yes"/>
+<layer number="28" name="bValues" color="7" fill="1" visible="no" active="yes"/>
 <layer number="29" name="tStop" color="7" fill="3" visible="no" active="yes"/>
 <layer number="30" name="bStop" color="7" fill="6" visible="no" active="yes"/>
@@
 <layer number="46" name="Milling" color="3" fill="1" visible="yes" active="yes"/>
 <layer number="47" name="Measures" color="7" fill="1" visible="yes" active="yes"/>
-<layer number="48" name="Document" color="7" fill="1" visible="no" active="yes"/>
-<layer number="49" name="Reference" color="7" fill="1" visible="no" active="yes"/>
+<layer number="48" name="Document" color="7" fill="1" visible="yes" active="yes"/>
+<layer number="49" name="Reference" color="7" fill="1" visible="yes" active="yes"/>
 <layer number="50" name="dxf" color="7" fill="1" visible="no" active="no"/>
-<layer number="51" name="tDocu" color="7" fill="1" visible="no" active="yes"/>
-<layer number="52" name="bDocu" color="7" fill="1" visible="yes" active="yes"/>
+<layer number="51" name="tDocu" color="7" fill="1" visible="yes" active="yes"/>
+<layer number="52" name="bDocu" color="7" fill="1" visible="no" active="yes"/>
 <layer number="53" name="tGND_GNDA" color="7" fill="9" visible="no" active="no"/>
 <layer number="54" name="bGND_GNDA" color="1" fill="9" visible="no" active="no"/>
@@
 <layer number="99" name="Anatomie" color="7" fill="1" visible="no" active="no"/>
 <layer number="100" name="Muster" color="7" fill="1" visible="no" active="no"/>
-<layer number="101" name="Hidden" color="57" fill="4" visible="no" active="yes"/>
-<layer number="102" name="Changes" color="13" fill="1" visible="no" active="yes"/>
+<layer number="101" name="Hidden" color="57" fill="4" visible="yes" active="yes"/>
+<layer number="102" name="Changes" color="13" fill="1" visible="yes" active="yes"/>
 <layer number="103" name="tMap" color="29" fill="4" visible="no" active="yes"/>
-<layer number="104" name="Name" color="16" fill="1" visible="no" active="yes"/>
+<layer number="104" name="Name" color="16" fill="1" visible="yes" active="yes"/>
 <layer number="105" name="tPlate" color="7" fill="1" visible="no" active="yes"/>
 <layer number="106" name="bPlate" color="7" fill="1" visible="no" active="yes"/>
@@
 <element name="R3X52" library="SPCoast" package="CUT-R" value="NOSTUFF" x="85.09" y="71.12" rot="R90"/>
 <element name="R4X52" library="SPCoast" package="CUT-R" value="NOSTUFF" x="82.55" y="71.12" rot="R90"/>
-<element name="CARRIER" library="SPCoast" package="BOARD-DINRAIL-3.17IN-5X2-IOP" value="" x="0" y="0"/>
-<element name="FID-UL" library="SPCoast" package="FIDUCIAL_1MM" value="" x="5.08" y="91.44" smashed="yes">
+<element name="CARRIER" library="SPCoast" package="BOARD-DINRAIL-3.17IN-5X2-IOP" value="10x10" x="0" y="0"/>
+<element name="FID-UL" library="SPCoast" package="FIDUCIAL_1MM" value="FIDUCIAL" x="5.08" y="91.44" smashed="yes">
 <attribute name="NAME" x="2.54" y="89.535" size="1.016" layer="25" rot="R90"/>
 </element>
-<element name="FID-LR" library="SPCoast" package="FIDUCIAL_1MM" value="" x="93.98" y="10.16" smashed="yes">
+<element name="FID-LR" library="SPCoast" package="FIDUCIAL_1MM" value="FIDUCIAL" x="93.98" y="10.16" smashed="yes">
 <attribute name="NAME" x="99.06" y="6.985" size="1.016" layer="25" rot="R90"/>
 </element>

Commit message: normalized values
Parts:
- CARRIER: value 10x10 -> BOARD
Changed lines of the file:
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@@
 <element name="R3X52" library="SPCoast" package="CUT-R" value="NOSTUFF" x="85.09" y="71.12" rot="R90"/>
 <element name="R4X52" library="SPCoast" package="CUT-R" value="NOSTUFF" x="82.55" y="71.12" rot="R90"/>
-<element name="CARRIER" library="SPCoast" package="BOARD-DINRAIL-3.17IN-5X2-IOP" value="10x10" x="0" y="0"/>
+<element name="CARRIER" library="SPCoast" package="BOARD-DINRAIL-3.17IN-5X2-IOP" value="BOARD" x="0" y="0"/>
 <element name="FID-UL" library="SPCoast" package="FIDUCIAL_1MM" value="FIDUCIAL" x="5.08" y="91.44" smashed="yes">
 <attribute name="NAME" x="2.54" y="89.535" size="1.016" layer="25" rot="R90"/>
